Commit message: Add files via upload

File: src/jettank/robot.urdf (robot description, URDF)
Before this commit: robot Jet_Tank, 7 links, 6 joints
Links:
- removed link imu_sensor
- link base_link: geometry collision box size=0.135 0.08 0.05; visual box size=0.135 0.08 0.05
- link camera: geometry collision box size=0.01 0.03 0.01; visual box size=0.01 0.03 0.01
- link omniwheel: geometry collision sphere radius=0.02; visual sphere radius=0.02
- link wheel_left: geometry collision cylinder length=0.02 radius=0.0325; visual cylinder length=0.02 radius=0.0325
- link wheel_right: geometry collision cylinder length=0.02 radius=0.033; visual cylinder length=0.02 radius=0.033
Joints:
- removed joint base_link_to_imu_sensor
- removed joint omniwheel_to_wheel_right
- added joint base_link_to_wheel_right: type continuous, parent base_link, child wheel_right, origin xyz=0.035 0.05 -0.005 rpy=1.5707963267948963 0 0, axis 0 0 1
- joint base_joint: origin xyz=0 0 0.5 rpy=0 0 0 -> xyz=0 0 0.05 rpy=0 0 0
- joint base_link_to_camera: origin xyz=1.6256258584357346 -0.02298885073006307 0.3695319117946291 rpy=0 0 0 -> xyz=0.06 0 0.03 rpy=0 0 0
- joint base_link_to_omniwheel: origin xyz=-1.3060831793408325 0 -0.3305897092162815 rpy=0 0 0 -> xyz=-0.045 0 -0.015 rpy=0 0 0
- joint base_link_to_wheel_left: origin xyz=1.39430638208543 -1.1736814480844906 -0.2208471930668996 rpy=1.5707963267948963 0 0 -> xyz=0.035 -0.05 -0.005 rpy=1.5707963267948963 0 0
